Commit message: Linked robotiq gripper package with ur5

File: robotiq_2f_85_gripper_visualization/urdf/robotiq_arg2f.xacro (robot description, xacro)
@@ -1,5 +1,12 @@
 <?xml version="1.0"?>
 <robot xmlns:xacro="http://ros.org/wiki/xacro">
-  <xacro:macro name="robotiq_arg2f_base_link" params="prefix">
+  <xacro:macro name="robotiq_arg2f_base_link" params="prefix connected_to">
+    <joint name="${prefix}_tool_joint" type="fixed">
+      <!-- The parent link must be read from the robot model it is attached to. -->
+      <parent link="${connected_to}"/>
+      <child link="${prefix}robotiq_arg2f_base_link"/>
+      <!-- The tool is directly attached to the flange. -->
+      <origin rpy="0 0 0" xyz="0 0 0"/>
+    </joint>
     <link name="${prefix}robotiq_arg2f_base_link">
       <inertial>

File: robotiq_2f_85_gripper_visualization/urdf/robotiq_arg2f_85_model.xacro (robot description, xacro)
@@ -2,4 +2,4 @@
 <robot name="robotiq_arg2f_85_model" xmlns:xacro="http://ros.org/wiki/xacro">
   <xacro:include filename="$(find robotiq_2f_85_gripper_visualization)/urdf/robotiq_arg2f_85_model_macro.xacro" />
-  <xacro:robotiq_arg2f_85 prefix=""/>
+  <xacro:robotiq_arg2f_85 prefix="" connected_to="world"/>
 </robot>

File: robotiq_2f_85_gripper_visualization/urdf/robotiq_arg2f_85_model_macro.xacro (robot description, xacro)
@@ -181,6 +181,7 @@
   </xacro:macro>
   <!-- Initialization of all joints and links -->
-  <xacro:macro name="robotiq_arg2f_85" params="prefix">
-    <xacro:robotiq_arg2f_base_link prefix="${prefix}"/>
+  <!-- CHANGES -->
+  <xacro:macro name="robotiq_arg2f_85" params="prefix connected_to">
+    <xacro:robotiq_arg2f_base_link prefix="${prefix}" connected_to="${connected_to}"/>
     <xacro:finger_links prefix="${prefix}" fingerprefix="left" stroke="85"/>
     <xacro:finger_links prefix="${prefix}" fingerprefix="right" stroke="85"/>
@@ -190,2 +191,3 @@
   </xacro:macro>
 </robot>
+<!-- CHANGES END -->
